Commit message: 0.4

File: src/my_robot_description/urdf/robot.urdf.xacro (robot description, xacro)
@@ -2,18 +2,26 @@
 <robot xmlns:xacro="http://www.ros.org/wiki/xacro" name="telega">
   <!-- ==================== Properties ==================== -->
-  <xacro:property name="base_length" value="0.6"/>
-  <xacro:property name="base_width" value="0.3"/>
-  <xacro:property name="base_height" value="0.2"/>
-  <xacro:property name="wheel_radius" value="0.035"/>
-  <xacro:property name="wheel_length" value="0.035"/>
-  <xacro:property name="base_mass" value="5.0"/>
-  <xacro:property name="wheel_mass" value="0.5"/>
+  <!-- Размеры корпуса робота (в метрах) -->
+  <xacro:property name="base_length" value="0.24"/>       <!-- Длина корпуса по оси X (от переднего до заднего края), м -->
+  <xacro:property name="base_width" value="0.17"/>        <!-- Ширина корпуса по оси Y (от левого до правого борта), м -->
+  <xacro:property name="base_height" value="0.11"/>       <!-- Высота корпуса по оси Z (от верха до низа), м -->
+  <!-- Параметры гусеницы (в метрах) -->
+  <xacro:property name="track_radius" value="0.0225"/>     <!-- Радиус катков и ведущего колеса, м -->
+  <xacro:property name="track_width" value="0.044"/>     <!-- Ширина гусеничной ленты, м -->
+  <xacro:property name="track_length" value="0.21"/>      <!-- Длина гусеницы (зона контакта с землёй), м -->
+  <!-- Массы компонентов (в кг) -->
+  <xacro:property name="base_mass" value="1.067"/>         <!-- Масса корпуса, кг -->
+  <xacro:property name="track_mass" value="0.030"/>        <!-- Масса одной гусеницы (лента), кг -->
+  <xacro:property name="roller_mass" value="0.012"/>       <!-- Масса одного катка, кг -->
+  <!-- Расстояние от центра катков до низа корпуса, м -->
+  <xacro:property name="roller_to_base_gap" value="0.014"/>
   <!-- ==================== Macros ==================== -->
-  <xacro:macro name="wheel_link" params="name">
+  <!-- Макрос: отдельный каток (визуал + коллизия + инерция) -->
+  <xacro:macro name="roller_link" params="name">
     <link name="${name}">
       <visual>
-        <origin rpy="1.57075 0 0" xyz="0 0 0"/>
+        <origin rpy="1.57075 0 0" xyz="0 0 0"/>       <!-- Поворот на 90° вокруг X, чтобы цилиндр лежал горизонтально -->
         <geometry>
-          <cylinder length="${wheel_length}" radius="${wheel_radius}"/>
+          <cylinder length="${track_width}" radius="${track_radius}"/>
         </geometry>
         <material name="dark_gray"/>
@@ -22,33 +30,85 @@
         <origin rpy="1.57075 0 0" xyz="0 0 0"/>
         <geometry>
-          <cylinder length="${wheel_length}" radius="${wheel_radius}"/>
+          <cylinder length="${track_width}" radius="${track_radius}"/>
         </geometry>
       </collision>
       <inertial>
-        <mass value="${wheel_mass}"/>
-        <inertia ixx="0.001" ixy="0.0" ixz="0.0" iyy="0.001" iyz="0.0" izz="0.001"/>
+        <mass value="${roller_mass}"/>                  <!-- Масса одного катка -->
+        <!-- Моменты инерции катка (упрощённо) -->
+        <inertia ixx="0.0005" ixy="0.0" ixz="0.0" iyy="0.0005" iyz="0.0" izz="0.0005"/>
       </inertial>
     </link>
   </xacro:macro>
-  <xacro:macro name="wheel_joint" params="name parent x y z">
-    <joint name="${name}_joint" type="continuous">
+  <!-- Макрос: сустав для катка (непрерывное вращение) -->
+  <xacro:macro name="roller_joint" params="name parent x y z">
+    <joint name="${name}_joint" type="continuous">    <!-- continuous = каток может вращаться бесконечно -->
       <parent link="${parent}"/>
       <child link="${name}"/>
-      <origin rpy="0 0 0" xyz="${x} ${y} ${z}"/>
-      <axis xyz="0 1 0"/>
+      <origin rpy="0 0 0" xyz="${x} ${y} ${z}"/>     <!-- Позиция катка относительно родительского link -->
+      <axis xyz="0 1 0"/>                              <!-- Ось вращения — по оси Y -->
     </joint>
   </xacro:macro>
+  <!-- Макрос: полная сборка гусеницы (левая или правая) -->
+  <xacro:macro name="track_assembly" params="side y_offset">
+    <!-- side   = "left" или "right" (какая гусеница) -->
+    <!-- y_offset = смещение по оси Y (расстояние от центра корпуса до центра гусеницы) -->
+    <!-- Гусеничная лента (визуальный прямоугольник, имитирует резиновое полотно) -->
+    <link name="${side}_track">
+      <visual>
+        <origin xyz="0 0 0" rpy="0 0 0"/>
+        <geometry>
+          <box size="${track_length} ${track_width} ${track_radius * 2 + 0.01}"/>  <!-- длина × ширина × высота -->
+        </geometry>
+        <material name="dark_gray"/>
+      </visual>
+      <collision>
+        <origin xyz="0 0 0" rpy="0 0 0"/>
+        <geometry>
+          <box size="${track_length} ${track_width} ${track_radius * 2 + 0.01}"/>
+        </geometry>
+      </collision>
+      <inertial>
+        <mass value="${track_mass}"/>                   <!-- Масса гусеничной ленты -->
+        <inertia ixx="0.01" ixy="0.0" ixz="0.0" iyy="0.01" iyz="0.0" izz="0.01"/>
+      </inertial>
+    </link>
+    <!-- Фиксированный сустав: приклеивает гусеничную ленту к корпусу -->
+    <joint name="${side}_track_joint" type="fixed">
+      <parent link="base_link"/>
+      <child link="${side}_track"/>
+      <origin xyz="0 ${y_offset} ${-base_height/2 - roller_to_base_gap}" rpy="0 0 0"/>  <!-- Гусеничная лента на уровне центров катков -->
+    </joint>
+    <!-- ===== Колёса и катки гусеницы ===== -->
+    <!-- Ведущее колесо (заднее) — крутит гусеницу -->
+    <xacro:roller_link name="${side}_drive_wheel"/>
+    <xacro:roller_joint name="${side}_drive_wheel" parent="base_link"
+                        x="-0.095" y="${y_offset}" z="${-base_height/2 - roller_to_base_gap}"/>
+    <!-- Поддерживающий каток #1 (передний) -->
+    <xacro:roller_link name="${side}_support_roller_1"/>
+    <xacro:roller_joint name="${side}_support_roller_1" parent="base_link"
+                        x="0.1" y="${y_offset}" z="${-base_height/2 - roller_to_base_gap}"/>
+    <!-- Поддерживающий каток #2 (центральный) -->
+    <xacro:roller_link name="${side}_support_roller_2"/>
+    <xacro:roller_joint name="${side}_support_roller_2" parent="base_link"
+                        x="0.04" y="${y_offset}" z="${-base_height/2 - roller_to_base_gap}"/>
+    <!-- Поддерживающий каток #3 (между центром и ведущим) -->
+    <xacro:roller_link name="${side}_support_roller_3"/>
+    <xacro:roller_joint name="${side}_support_roller_3" parent="base_link"
+                        x="-0.035" y="${y_offset}" z="${-base_height/2 - roller_to_base_gap}"/>
+  </xacro:macro>
   <!-- ==================== Materials ==================== -->
+  <!-- Цвета для визуализации в RViz (R, G, B, Alpha — от 0.0 до 1.0) -->
   <material name="blue">
-    <color rgba="0.2 0.4 0.8 1.0"/>
+    <color rgba="0.2 0.4 0.8 1.0"/>                    <!-- Синий цвет для корпуса -->
   </material>
   <material name="dark_gray">
-    <color rgba="0.3 0.3 0.3 1.0"/>
+    <color rgba="0.3 0.3 0.3 1.0"/>                    <!-- Тёмно-серый для гусениц и катков -->
   </material>
   <!-- ==================== Base Link ==================== -->
+  <!-- Основной корпус робота (прямоугольный параллелепипед) -->
   <link name="base_link">
     <visual>
       <geometry>
-        <box size="${base_length} ${base_width} ${base_height}"/>
+        <box size="${base_length} ${base_width} ${base_height}"/>  <!-- Длина × Ширина × Высота -->
       </geometry>
       <material name="blue"/>
@@ -56,27 +116,18 @@
     <collision>
       <geometry>
-        <box size="${base_length} ${base_width} ${base_height}"/>
+        <box size="${base_length} ${base_width} ${base_height}"/>  <!-- Границы для обнаружения столкновений -->
       </geometry>
     </collision>
     <inertial>
-      <mass value="${base_mass}"/>
+      <mass value="${base_mass}"/>                       <!-- Масса корпуса, кг -->
+      <!-- Моменты инерции корпуса (упрощённо, для прямоугольника) -->
       <inertia ixx="0.05" ixy="0.0" ixz="0.0" iyy="0.05" iyz="0.0" izz="0.05"/>
     </inertial>
   </link>
-  <!-- ==================== Wheels ==================== -->
-  <!-- Left wheels -->
-  <xacro:wheel_link name="left_front_wheel"/>
-  <xacro:wheel_link name="left_back_wheel"/>
-  <!-- Right wheels -->
-  <xacro:wheel_link name="right_front_wheel"/>
-  <xacro:wheel_link name="right_back_wheel"/>
-  <!-- Wheel joints -->
-  <xacro:wheel_joint name="left_front_wheel" parent="base_link"
-                     x="${base_length/2 - 0.1}" y="${base_width/2 + wheel_length/2}" z="${-base_height/2 - wheel_radius + 0.01}"/>
-  <xacro:wheel_joint name="left_back_wheel" parent="base_link"
-                     x="${-base_length/2 + 0.1}" y="${base_width/2 + wheel_length/2}" z="${-base_height/2 - wheel_radius + 0.01}"/>
-  <xacro:wheel_joint name="right_front_wheel" parent="base_link"
-                     x="${base_length/2 - 0.1}" y="${-base_width/2 - wheel_length/2}" z="${-base_height/2 - wheel_radius + 0.01}"/>
-  <xacro:wheel_joint name="right_back_wheel" parent="base_link"
-                     x="${-base_length/2 + 0.1}" y="${-base_width/2 - wheel_length/2}" z="${-base_height/2 - wheel_radius + 0.01}"/>
+  <!-- ==================== Tracks ==================== -->
+  <!-- Установка двух гусениц: левая и правая -->
+  <!-- Левая гусеница: смещена вправо от центра (base_width/2) на половину ширины гусеницы -->
+  <xacro:track_assembly side="left" y_offset="${base_width/2 + track_width/2}"/>
+  <!-- Правая гусеница: смещена влево от центра (-base_width/2) на половину ширины гусеницы -->
+  <xacro:track_assembly side="right" y_offset="${-base_width/2 - track_width/2}"/>
 </robot>

Commit message: feat: add MaixSense A10 ToF camera to robot description and optimize launch GUI check

File: src/my_robot_description/urdf/robot.urdf.xacro (robot description, xacro)
@@ -131,3 +131,48 @@
   <!-- Правая гусеница: смещена влево от центра (-base_width/2) на половину ширины гусеницы -->
   <xacro:track_assembly side="right" y_offset="${-base_width/2 - track_width/2}"/>
+  <!-- ==================== MaixSense A010 ToF Camera ==================== -->
+  <!-- Свойства камеры -->
+  <xacro:property name="tof_length" value="0.01"/>       <!-- Глубина (X), м (10 мм) -->
+  <xacro:property name="tof_width" value="0.034"/>       <!-- Ширина (Y), м (34 мм) -->
+  <xacro:property name="tof_height" value="0.023"/>      <!-- Высота (Z), м (23 мм) -->
+  <xacro:property name="tof_mass" value="0.010"/>        <!-- Масса 10 г -->
+  <!-- Гармоничный цвет для корпуса камеры (малиновый/черри) -->
+  <material name="crimson">
+    <color rgba="0.8 0.1 0.2 1.0"/>
+  </material>
+  <!-- Физический корпус камеры -->
+  <link name="tof_link">
+    <visual>
+      <origin xyz="0 0 0" rpy="0 0 0"/>
+      <geometry>
+        <box size="${tof_length} ${tof_width} ${tof_height}"/>
+      </geometry>
+      <material name="crimson"/>
+    </visual>
+    <collision>
+      <origin xyz="0 0 0" rpy="0 0 0"/>
+      <geometry>
+        <box size="${tof_length} ${tof_width} ${tof_height}"/>
+      </geometry>
+    </collision>
+    <inertial>
+      <mass value="${tof_mass}"/>
+      <inertia ixx="0.000001" ixy="0.0" ixz="0.0" iyy="0.000001" iyz="0.0" izz="0.000001"/>
+    </inertial>
+  </link>
+  <!-- Крепление камеры на переднем торце корпуса, по центру по Y и приподнято по Z (повернуто боком на 90 градусов по X) -->
+  <joint name="tof_joint" type="fixed">
+    <parent link="base_link"/>
+    <child link="tof_link"/>
+    <origin xyz="${base_length/2 + tof_length/2} 0 0.04" rpy="1.57079632679 0 0"/>
+  </joint>
+  <!-- Оптический кадр (frame_id для топиков ROS 2 depth и cloud) -->
+  <link name="tof"/>
+  <!-- Переход от стандартных координат робота к оптическим координатам камеры -->
+  <!-- Привязан напрямую к base_link для сохранения стандартной (неповернутой) ориентации данных -->
+  <joint name="tof_optical_joint" type="fixed">
+    <parent link="base_link"/>
+    <child link="tof"/>
+    <origin xyz="${base_length/2 + tof_length/2} 0 0.04" rpy="-1.57079632679 0 -1.57079632679"/>
+  </joint>
 </robot>
